Commit message: feat: correct pebbles urdf + soft limits joints

File: earth_moving/clutter/urdf/pebbles/pebbles.urdf (robot description, URDF)
Before this commit: robot shovel, 2 links, 1 joints
Links:
- removed link base_link
Joints:
- removed joint base_pebbles_joint

File: earth_moving/clutter/urdf/shovel/shovelFlat.urdf (robot description, URDF)
Before this commit: robot shovel, 3 links, 2 joints
Joints:
- joint shovel_shadow_joint: limit lower=-0.2 upper=0.2 effort=1e2 velocity=3.1415 -> lower=-0.2 upper=0.2 effort=1e2 velocity=1
