Commit message: chore: simple flat moving

File: earth_moving/clutter/urdf/shovel/shovelFlat.urdf (robot description, URDF)
Before this commit: robot shovel, 3 links, 2 joints
Links:
- removed link shadow_link
Joints:
- removed joint shovel_shadow_joint

Commit message: chore: engine.py class

File: earth_moving/clutter/urdf/shovel/shovelFlat.urdf (robot description, URDF)
Before this commit: robot shovel, 2 links, 1 joints
Links:
- added link shadow_link, mass 20e-3; collision box size=1e-2 1e-1 5e-2; visual box size=1e-2 1e-1 5e-2
Joints:
- added joint shovel_shadow_joint: type revolute, parent shovel_link, child shadow_link, origin xyz=0.05 0 0 rpy=0 0 0, axis 0 0 1, limit lower=-3.1415/12 upper=3.1415/12 effort=1e2 velocity=3.1415

Commit message: dev: trying to solve the compenetration issue

File: earth_moving/clutter/urdf/shovel/shovelFlat.urdf (robot description, URDF)
Before this commit: robot shovel, 3 links, 2 joints
Joints:
- joint shovel_shadow_joint: limit lower=-3.1415/12 upper=3.1415/12 effort=1e2 velocity=3.1415 -> lower=-0.2 upper=0.2 effort=1e2 velocity=3.1415

Commit message: feat: PRR urdf

File: earth_moving/clutter/urdf/shovel/shovelFlat.urdf (robot description, URDF)
Before this commit: robot shovel, 3 links, 2 joints
Links:
- removed link shadow_link
- removed link shovel_link
- added link EE_link, mass 20e-3; collision box size=1e-2 1e-1 5e-2; visual box size=1e-2 1e-1 5e-2
- added link L1_link, mass 20e-3; collision box size=5e-2 1e-2 5e-2; visual box size=1e-1 5e-2 5e-2
- added link L2_link, mass 0.0; collision cylinder length=1e-1 radius=1e-2; visual cylinder length=1e-1 radius=1e-2
Joints:
- removed joint base_shovel_joint
- removed joint shovel_shadow_joint
- added joint L1_L2_joint: type revolute, parent L1_link, child L2_link, origin xyz=1e-1 0 0 rpy=0 0 0, axis 0 0 1, limit lower=-3.1415 upper=3.1415 effort=1e2 velocity=0.2
- added joint L2_EE_joint: type revolute, parent L2_link, child EE_link, origin xyz=5e-2 0 0 rpy=0 0 0, axis 0 0 1, limit lower=-0.2 upper=0.2 effort=1e2 velocity=1
- added joint base_L1_joint: type prismatic, parent base_link, child L1_link, origin xyz=5e-1 0 2.5e-2 rpy=0 0 0, axis 1 0 0, limit lower=-10 upper=10 effort=1e2 velocity=0.2

Commit message: dev: position and vel control

File: earth_moving/clutter/urdf/shovel/shovelFlat.urdf (robot description, URDF)
Before this commit: robot shovel, 4 links, 3 joints
Joints:
- joint L1_L2_joint: limit lower=-3.1415 upper=3.1415 effort=1e2 velocity=0.2 -> lower=-3.1415 upper=3.1415 effort=1e2 velocity=0.01
- joint L2_EE_joint: limit lower=-0.2 upper=0.2 effort=1e2 velocity=1 -> lower=-1.57 upper=1.57 effort=1e2 velocity=0.01; origin xyz=5e-2 0 0 rpy=0 0 0 -> xyz=1e-1 0 0 rpy=0 0 0

Commit message: dev: ok with vel control, not so good with position. TODO: control all joints together

File: earth_moving/clutter/urdf/shovel/shovelFlat.urdf (robot description, URDF)
Before this commit: robot shovel, 4 links, 3 joints
Joints:
- joint L1_L2_joint: limit lower=-3.1415 upper=3.1415 effort=1e2 velocity=0.01 -> lower=-3.1415 upper=3.1415 effort=1e2 velocity=0.2
- joint L2_EE_joint: limit lower=-1.57 upper=1.57 effort=1e2 velocity=0.01 -> lower=-1.57 upper=1.57 effort=1e2 velocity=0.2
- joint base_L1_joint: limit lower=-10 upper=10 effort=1e2 velocity=0.2 -> lower=-10 upper=10 effort=1e2 velocity=0.5

Commit message: fix: controlMotorArray instead of MultiDof

File: earth_moving/clutter/urdf/shovel/shovelFlat.urdf (robot description, URDF)
Before this commit: robot shovel, 4 links, 3 joints
Links:
- link L2_link: geometry collision cylinder length=1e-1 radius=1e-2; visual cylinder length=5.1e-2 radius=4e-2
Joints:
- joint L1_L2_joint: origin xyz=1e-1 0 0 rpy=0 0 0 -> xyz=0 0 0 rpy=0 0 0
- joint L2_EE_joint: origin xyz=1e-1 0 0 rpy=0 0 0 -> xyz=2e-1 0 0 rpy=0 0 0
