Commit message: Add envs and gym enviroment

File: earth_moving/clutter/urdf/shovel/rover_with_shovel.urdf (robot description, URDF)
Before this commit: robot test_robot, 6 links, 5 joints
Links:
- link base_link: geometry collision box size=0.32 0.17 0.05; visual box size=0.32 0.17 0.05
- link lwheel: geometry collision cylinder length=0.008 radius=0.07; visual cylinder length=0.008 radius=0.07
- link lwheel_back: geometry collision cylinder length=0.008 radius=0.07; visual cylinder length=0.008 radius=0.07
- link rwheel: geometry collision cylinder length=0.008 radius=0.07; visual cylinder length=0.008 radius=0.07
- link rwheel_back: geometry collision cylinder length=0.008 radius=0.07; visual cylinder length=0.008 radius=0.07
- link shovel: geometry collision box size=0.01 0.22 0.08; visual box size=0.01 0.22 0.08
Joints:
- joint base_to_fattach: origin xyz=0.08 0 0.025 rpy=0 0 0 -> xyz=0.17 0 0.042 rpy=0 0 0
- joint base_to_lwheel: origin xyz=0.035 0.045 0.026 rpy=1.5708 0 0 -> xyz=0.08 0.1 0.07 rpy=1.5708 0 0
- joint base_to_lwheel_back: origin xyz=-0.035 0.045 0.026 rpy=1.5708 0 0 -> xyz=-0.08 0.1 0.07 rpy=1.5708 0 0
- joint base_to_rwheel: origin xyz=0.035 -0.045 0.026 rpy=1.5708 0 0 -> xyz=0.08 -0.1 0.07 rpy=1.5708 0 0
- joint base_to_rwheel_back: origin xyz=-0.0350 -0.045 0.026 rpy=1.5708 0 0 -> xyz=-0.080 -0.1 0.07 rpy=1.5708 0 0
