Commit message: 2 wheel rover

File: earth_moving/clutter/urdf/shovel/2_wheel_rover.urdf (robot description, URDF)
Before this commit: robot test_robot, 4 links, 3 joints
Links:
- added link shovel, mass 0.3; collision box size=0.01 0.22 0.08; visual box size=0.01 0.22 0.08
Joints:
- added joint base_to_fattach: type fixed, parent base_link, child shovel, origin xyz=0.17 0 0.042 rpy=0 0 0

Commit message: chore: test urdf

File: earth_moving/clutter/urdf/shovel/2_wheel_rover.urdf (robot description, URDF)
Before this commit: robot test_robot, 5 links, 4 joints
Joints:
- removed joint base_to_fattach
- added joint base_to_shovel: type prismatic, parent base_link, child shovel, origin xyz=0.17 0 0.042 rpy=0 0 0, axis 1 0 0, limit lower=0.0 upper=0.1 effort=50 velocity=0.1
