Commit message: fix: deadzone stuck control

File: earth_moving/3d integration/2_wheel_rover.urdf (robot description, URDF)
Before this commit: robot test_robot, 5 links, 4 joints
Links:
- removed link front_wheel
- link base_link: geometry collision box size=0.20 0.17 0.05; visual box size=0.20 0.17 0.05
- link lwheel: geometry collision cylinder length=0.02 radius=0.05; visual cylinder length=0.02 radius=0.05
- link rwheel: geometry collision cylinder length=0.02 radius=0.05; visual cylinder length=0.02 radius=0.05
- link shovel: geometry collision box size=0.01 0.22 0.06; visual box size=0.01 0.22 0.06
Joints:
- removed joint base_to_front_wheel
- joint base_to_fattach: origin xyz=0.17 0 0.042 rpy=0 0 0 -> xyz=0.11 0 0.042 rpy=0 0 0
- joint base_to_lwheel: origin xyz=-0.12 0.1 0.07 rpy=1.5708 0 0 -> xyz=-0.06 0.1 0.05 rpy=1.5708 0 0
- joint base_to_rwheel: origin xyz=-0.12 -0.1 0.07 rpy=1.5708 0 0 -> xyz=-0.06 -0.1 0.05 rpy=1.5708 0 0
