Commit message: feat: working velocity control

File: earth_moving/clutter/shovel/urdf/pebbles/pebbles.urdf (robot description, URDF)
Before this commit: robot shovel, 1 links, 0 joints
Links:
- link pebbles_link: geometry collision box size=2e-2 2e-2 2e-2; visual box size=2e-2 2e-2 2e-2

File: earth_moving/clutter/shovel/urdf/shovel/shovelFlat.urdf (robot description, URDF)
Before this commit: robot shovel, 4 links, 3 joints
Links:
- link EE_link: geometry collision box size=1e-2 2e-1 5e-2; visual box size=1e-2 2e-1 5e-2
- link base_link: mass 1e-3 -> 1e4; geometry collision box size=0.1 0.1 0.1; visual box size=0.1 0.1 0.1
Joints:
- joint L1_L2_joint: limit lower=-10 upper=10 effort=1e2 velocity=0.005 -> lower=-10 upper=10 effort=1e2 velocity=0.5; origin xyz=0 0 0 rpy=0 0 0 -> xyz=0.1 0 0.1 rpy=0 0 0
- joint L2_EE_joint: limit lower=-3.14159 upper=3.14159 effort=1e2 velocity=0.005 -> lower=-3.14159 upper=3.14159 effort=1e2 velocity=0.5; origin xyz=0 0 0 rpy=0 0 0 -> xyz=0.1 0 -0.225 rpy=0 0 0
- joint base_L1_joint: limit lower=-10 upper=10 effort=1e2 velocity=0.005 -> lower=-10 upper=10 effort=1e2 velocity=0.5; origin xyz=0 0 0 rpy=0 0 0 -> xyz=-0.2 0 0.1 rpy=0 0 0
